Commit message: update urdf

File: catkin_ws/src/roomba/roomba_description/urdf/roomba.urdf.xacro (robot description, xacro)
@@ -1,36 +1,24 @@
 <?xml version="1.0"?>
 <robot name="roomba" xmlns:xacro="http://ros.org/wiki/xacro">
-  <xacro:include filename="$(find create_description)/urdf/create_base.urdf.xacro" />
-  <xacro:include filename="$(find create_description)/urdf/create_2_gazebo.urdf.xacro" />
-  <xacro:create_base wheel_separation="0.235" base_diameter="0.3485">
-    <mesh filename="package://create_description/meshes/create_2.dae" />
-  </xacro:create_base>
-  <link name="lidar_base">
+  <link name="base_link">
     <inertial>
-      <origin xyz="0 0 0" rpy="0 0 0"/>
-      <mass value="0.5"/>
+      <origin xyz="0 0 0" rpy="1.57 0 1.57" />
+      <mass value="1.0"/>
       <inertia ixx="100"  ixy="0"  ixz="0" iyy="100" iyz="0" izz="100" />
     </inertial>
     <visual>
-      <origin xyz="0 0 0" rpy="0 0 0" />
+      <origin xyz="0 0 0" rpy="1.57 0 1.57" />
       <geometry>
-        <box size="0.09 0.12 0.05" />
+        <mesh filename="package://roomba_description/meshes/roomba_hack.stl" scale="0.001 0.001 0.001" />
       </geometry>
-      <material name="white">
-          <color rgba="1.0 1.0 1.0 1.0"/>
-      </material>
+      <material name="grey"/>
     </visual>
     <collision>
-      <origin xyz="0 0 0" rpy="0 0 0" />
+      <origin xyz="0 0 0" rpy="1.57 0 1.57" />
       <geometry>
-        <box size="0.09 0.12 0.05" />
+        <mesh filename="package://roomba_description/meshes/roomba_hack.stl" scale="0.001 0.001 0.001" />
       </geometry>
     </collision>
   </link>
-  <joint name="lidar_base_to_base_link" type="fixed">
-    <origin xyz="0.09 0 0.09" rpy="0 0 0"/>
-    <parent link="base_link"/>
-    <child link="lidar_base"/>
-  </joint>
   <link name="rplidar">
     <inertial>
@@ -54,65 +42,7 @@
   </link>
   <joint name="rplidar_to_base_link" type="fixed">
-    <origin xyz="0.05 0.0 0.0" rpy="0 0 0"/>
-    <parent link="lidar_base"/>
+    <origin xyz="-0.05 0.0 0.25" rpy="0 0 3.14"/>
+    <parent link="base_link"/>
     <child link="rplidar"/>
   </joint>
-  <link name="laser"/>
-  <joint name="laser_to_rplidar" type="fixed">
-    <origin xyz="-0.035 0.0 0.045" rpy="0 0 3.14159"/>
-    <parent link="rplidar"/>
-    <child link="laser"/>
-  </joint>
-  <link name="mobile_battery">
-    <inertial>
-      <origin xyz="0 0 0" rpy="0 0 0"/>
-      <mass value="0.680389"/>
-      <inertia ixx="100"  ixy="0"  ixz="0" iyy="100" iyz="0" izz="100" />
-    </inertial>
-    <visual>
-      <origin xyz="0 0 0" rpy="0 0 0" />
-      <geometry>
-        <box size="0.06 0.1 0.02" />
-      </geometry>
-      <material name="white">
-          <color rgba="1.0 1.0 1.0 1.0"/>
-      </material>
-    </visual>
-    <collision>
-      <origin xyz="0 0 0" rpy="0 0 0" />
-      <geometry>
-        <box size="0.06 0.1 0.02" />
-      </geometry>
-    </collision>
-  </link>
-  <joint name="mobile_battery_to_base_link" type="fixed">
-    <origin xyz="0.0 0.0 0.09" rpy="0 1.570796 0"/>
-    <parent link="base_link"/>
-    <child link="mobile_battery"/>
-  </joint>
-  <link name="jetson_nano">
-    <inertial>
-      <origin xyz="0 0 0" rpy="0 0 0"/>
-      <mass value="1.548"/>
-      <inertia ixx="100"  ixy="0"  ixz="0" iyy="100" iyz="0" izz="100" />
-    </inertial>
-    <visual>
-      <origin xyz="0 0 0" rpy="0 0 0" />
-      <geometry>
-        <box size="0.105 0.105 0.065" />
-      </geometry>
-      <material name="grey"/>
-    </visual>
-    <collision>
-      <origin xyz="0 0 0" rpy="0 0 0" />
-      <geometry>
-        <box size="0.105 0.105 0.065" />
-      </geometry>
-    </collision>
-  </link>
-  <joint name="jetson_nano_to_base_link" type="fixed">
-    <origin xyz="-0.1 0 0.09" rpy="0 0 0"/>
-    <parent link="base_link"/>
-    <child link="jetson_nano"/>
-  </joint>
 </robot>

Commit message: add laser link

File: catkin_ws/src/roomba/roomba_description/urdf/roomba.urdf.xacro (robot description, xacro)
@@ -46,3 +46,9 @@
     <child link="rplidar"/>
   </joint>
+  <link name="laser"/>
+  <joint name="laser_to_rplidar" type="fixed">
+    <origin xyz="0 0 0" rpy="0 0 3.14"/>
+    <parent link="rplidar"/>
+    <child link="laser"/>
+  </joint>
 </robot>

Commit message: update urdf

File: catkin_ws/src/roomba/roomba_description/urdf/roomba.urdf.xacro (robot description, xacro)
@@ -1,24 +1,36 @@
 <?xml version="1.0"?>
 <robot name="roomba" xmlns:xacro="http://ros.org/wiki/xacro">
-  <link name="base_link">
+  <xacro:include filename="$(find create_description)/urdf/create_base.urdf.xacro"/>
+  <xacro:include filename="$(find create_description)/urdf/create_2_gazebo.urdf.xacro"/>
+  <xacro:create_base wheel_separation="0.235" base_diameter="0.3485">
+    <mesh filename="package://create_description/meshes/create_2.dae"/>
+  </xacro:create_base>
+  <link name="lidar_base">
     <inertial>
-      <origin xyz="0 0 0" rpy="1.57 0 1.57" />
+      <origin xyz="0 0 0" rpy="0 0 0"/>
       <mass value="1.0"/>
       <inertia ixx="100"  ixy="0"  ixz="0" iyy="100" iyz="0" izz="100" />
     </inertial>
     <visual>
-      <origin xyz="0 0 0" rpy="1.57 0 1.57" />
+      <origin xyz="0 0 0" rpy="0 0 0"/>
       <geometry>
-        <mesh filename="package://roomba_description/meshes/roomba_hack.stl" scale="0.001 0.001 0.001" />
+        <box size="0.14 0.14 0.12"/>
       </geometry>
-      <material name="grey"/>
+      <material name="white">
+        <color rgba="1.0 1.0 1.0 1.0"/>
+      </material>
     </visual>
     <collision>
-      <origin xyz="0 0 0" rpy="1.57 0 1.57" />
+      <origin xyz="0 0 0" rpy="0 0 0"/>
       <geometry>
-        <mesh filename="package://roomba_description/meshes/roomba_hack.stl" scale="0.001 0.001 0.001" />
+        <box size="0.14 0.14 0.12"/>
       </geometry>
     </collision>
   </link>
+  <joint name="lidar_base_to_base_link" type="fixed">
+    <origin xyz="0 0 0.09" rpy="0 0 0"/>
+    <parent link="base_link"/>
+    <child link="lidar_base"/>
+  </joint>
   <link name="rplidar">
     <inertial>
@@ -42,11 +54,11 @@
   </link>
   <joint name="rplidar_to_base_link" type="fixed">
-    <origin xyz="-0.05 0.0 0.25" rpy="0 0 3.14"/>
-    <parent link="base_link"/>
+    <origin xyz="-0.05 0.0 0.06" rpy="0 0 3.14"/>
+    <parent link="lidar_base"/>
     <child link="rplidar"/>
   </joint>
   <link name="laser"/>
   <joint name="laser_to_rplidar" type="fixed">
-    <origin xyz="0 0 0" rpy="0 0 3.14"/>
+    <origin xyz="-0.035 0 0.045" rpy="0 0 3.14"/>
     <parent link="rplidar"/>
     <child link="laser"/>

Commit message: update urdf

File: catkin_ws/src/roomba/roomba_description/urdf/roomba.urdf.xacro (robot description, xacro)
@@ -2,5 +2,6 @@
 <robot name="roomba" xmlns:xacro="http://ros.org/wiki/xacro">
   <xacro:include filename="$(find create_description)/urdf/create_base.urdf.xacro"/>
-  <xacro:include filename="$(find create_description)/urdf/create_2_gazebo.urdf.xacro"/>
+  <xacro:include filename="$(find roomba_description)/urdf/common.xacro"/>
+  <xacro:include filename="$(find roomba_description)/urdf/sensors/rplidar.urdf.xacro"/>
   <xacro:create_base wheel_separation="0.235" base_diameter="0.3485">
     <mesh filename="package://create_description/meshes/create_2.dae"/>
@@ -33,34 +34,13 @@
     <child link="lidar_base"/>
   </joint>
-  <link name="rplidar">
-    <inertial>
-      <origin xyz="0 0 0" rpy="0 0 0"/>
-      <mass value="0.190"/>
-      <inertia ixx="100"  ixy="0"  ixz="0" iyy="100" iyz="0" izz="100" />
-    </inertial>
-    <visual>
-      <origin xyz="0 -0.035 0" rpy="1.570796 0 3.14159" />
-      <geometry>
-        <mesh filename="package://roomba_description/meshes/rplidar.stl" scale="0.001 0.001 0.001" />
-      </geometry>
-      <material name="grey"/>
-    </visual>
-    <collision>
-      <origin xyz="0 -0.035 0" rpy="1.570796 0 3.14159" />
-      <geometry>
-        <mesh filename="package://roomba_description/meshes/rplidar.stl" scale="0.001 0.001 0.001" />
-      </geometry>
-    </collision>
-  </link>
-  <joint name="rplidar_to_base_link" type="fixed">
-    <origin xyz="-0.05 0.0 0.06" rpy="0 0 3.14"/>
-    <parent link="lidar_base"/>
-    <child link="rplidar"/>
-  </joint>
-  <link name="laser"/>
-  <joint name="laser_to_rplidar" type="fixed">
-    <origin xyz="-0.035 0 0.045" rpy="0 0 3.14"/>
-    <parent link="rplidar"/>
-    <child link="laser"/>
-  </joint>
+  <xacro:rplidar prefix="rplidar" parent="lidar_base">
+    <origin xyz="-0.05 0.0 0.06" rpy="0 0 ${PI}"/>
+  </xacro:rplidar>
+  <!-- Gazebo -->
+  <gazebo>
+    <plugin name="gazebo_ros_control" filename="libgazebo_ros_control.so">
+      <robotNamespace>/roomba</robotNamespace>
+    </plugin>
+  </gazebo>
+  <xacro:rplidar_gazebo prefix="rplidar" min_rad="${-PI}" max_rad="${PI}" min_range="0.15" max_range="6"/>
 </robot>

Commit message: change urdf

File: catkin_ws/src/roomba/roomba_description/urdf/roomba.urdf.xacro (robot description, xacro)
@@ -15,5 +15,5 @@
       <origin xyz="0 0 0" rpy="0 0 0" />
       <geometry>
-        <box size="0.09 0.12 0.05" />
+        <box size="0.1 0.12 0.09" />
       </geometry>
       <material name="white">
@@ -24,10 +24,10 @@
       <origin xyz="0 0 0" rpy="0 0 0" />
       <geometry>
-        <box size="0.09 0.12 0.05" />
+        <box size="0.1 0.12 0.09" />
       </geometry>
     </collision>
   </link>
   <joint name="lidar_base_to_base_link" type="fixed">
-    <origin xyz="0.09 0 0.09" rpy="0 0 0"/>
+    <origin xyz="-0.08 0 0.09" rpy="0 0 0"/>
     <parent link="base_link"/>
     <child link="lidar_base"/>
@@ -40,5 +40,5 @@
     </inertial>
     <visual>
-      <origin xyz="0 -0.035 0" rpy="1.570796 0 3.14159" />
+      <origin xyz="0 0 0" rpy="1.570796 0 3.141592" />
       <geometry>
         <mesh filename="package://roomba_description/meshes/rplidar.stl" scale="0.001 0.001 0.001" />
@@ -47,5 +47,5 @@
     </visual>
     <collision>
-      <origin xyz="0 -0.035 0" rpy="1.570796 0 3.14159" />
+      <origin xyz="0 0 0" rpy="1.570796 0 3.141592" />
       <geometry>
         <mesh filename="package://roomba_description/meshes/rplidar.stl" scale="0.001 0.001 0.001" />
@@ -54,5 +54,5 @@
   </link>
   <joint name="rplidar_to_base_link" type="fixed">
-    <origin xyz="0.05 0.0 0.0" rpy="0 0 0"/>
+    <origin xyz="0.05 -0.033 0.045" rpy="0 0 0"/>
     <parent link="lidar_base"/>
     <child link="rplidar"/>
@@ -64,4 +64,5 @@
     <child link="laser"/>
   </joint>
+  <!--
   <link name="mobile_battery">
     <inertial>
@@ -116,3 +117,4 @@
     <child link="jetson_nano"/>
   </joint>
+  -->
 </robot>

Commit message: add

File: catkin_ws/src/roomba/roomba_description/urdf/roomba.urdf.xacro (robot description, xacro)
@@ -53,4 +53,16 @@
     </collision>
   </link>
+  <link name="realsense">
+    <visual>
+      <geometry>
+        <mesh filename="package://roomba_description/meshes/d435.stl" />
+      </geometry>
+    </visual>
+  </link>
+  <joint name="realsense_to_base_link" type="fixed">
+    <origin xyz="0.05 -0.033 0.045" rpy="0 0 0"/>
+    <parent link="lidar_base"/>
+    <child link="realsense"/>
+  </joint>
   <joint name="rplidar_to_base_link" type="fixed">
     <origin xyz="0.05 -0.033 0.045" rpy="0 0 0"/>

Commit message: change for lec

File: catkin_ws/src/roomba/roomba_description/urdf/roomba.urdf.xacro (robot description, xacro)
@@ -1,46 +1,132 @@
 <?xml version="1.0"?>
 <robot name="roomba" xmlns:xacro="http://ros.org/wiki/xacro">
-  <xacro:include filename="$(find create_description)/urdf/create_base.urdf.xacro"/>
-  <xacro:include filename="$(find roomba_description)/urdf/common.xacro"/>
-  <xacro:include filename="$(find roomba_description)/urdf/sensors/rplidar.urdf.xacro"/>
+  <xacro:include filename="$(find create_description)/urdf/create_base.urdf.xacro" />
+  <xacro:include filename="$(find create_description)/urdf/create_2_gazebo.urdf.xacro" />
   <xacro:create_base wheel_separation="0.235" base_diameter="0.3485">
-    <mesh filename="package://create_description/meshes/create_2.dae"/>
+    <mesh filename="package://create_description/meshes/create_2.dae" />
   </xacro:create_base>
   <link name="lidar_base">
     <inertial>
       <origin xyz="0 0 0" rpy="0 0 0"/>
-      <mass value="1.0"/>
+      <mass value="0.5"/>
       <inertia ixx="100"  ixy="0"  ixz="0" iyy="100" iyz="0" izz="100" />
     </inertial>
     <visual>
-      <origin xyz="0 0 0" rpy="0 0 0"/>
+      <origin xyz="0 0 0" rpy="0 0 0" />
       <geometry>
-        <box size="0.14 0.14 0.12"/>
+        <box size="0.1 0.12 0.09" />
       </geometry>
       <material name="white">
-        <color rgba="1.0 1.0 1.0 1.0"/>
+          <color rgba="1.0 1.0 1.0 1.0"/>
       </material>
     </visual>
     <collision>
-      <origin xyz="0 0 0" rpy="0 0 0"/>
+      <origin xyz="0 0 0" rpy="0 0 0" />
       <geometry>
-        <box size="0.14 0.14 0.12"/>
+        <box size="0.1 0.12 0.09" />
       </geometry>
     </collision>
   </link>
   <joint name="lidar_base_to_base_link" type="fixed">
-    <origin xyz="0 0 0.09" rpy="0 0 0"/>
+    <origin xyz="-0.08 0 0.09" rpy="0 0 0"/>
     <parent link="base_link"/>
     <child link="lidar_base"/>
   </joint>
-  <xacro:rplidar prefix="rplidar" parent="lidar_base">
-    <origin xyz="-0.05 0.0 0.06" rpy="0 0 ${PI}"/>
-  </xacro:rplidar>
-  <!-- Gazebo -->
-  <gazebo>
-    <plugin name="gazebo_ros_control" filename="libgazebo_ros_control.so">
-      <robotNamespace>/roomba</robotNamespace>
-    </plugin>
-  </gazebo>
-  <xacro:rplidar_gazebo prefix="rplidar" min_rad="${-PI}" max_rad="${PI}" min_range="0.15" max_range="6"/>
+  <link name="rplidar">
+    <inertial>
+      <origin xyz="0 0 0" rpy="0 0 0"/>
+      <mass value="0.190"/>
+      <inertia ixx="100"  ixy="0"  ixz="0" iyy="100" iyz="0" izz="100" />
+    </inertial>
+    <visual>
+      <origin xyz="0 0 0" rpy="1.570796 0 3.141592" />
+      <geometry>
+        <mesh filename="$(find roomba_description)/meshes/rplidar.stl" scale="0.001 0.001 0.001" />
+      </geometry>
+      <material name="grey"/>
+    </visual>
+    <collision>
+      <origin xyz="0 0 0" rpy="1.570796 0 3.141592" />
+      <geometry>
+        <mesh filename="$(find roomba_description)/meshes/rplidar.stl" scale="0.001 0.001 0.001" />
+      </geometry>
+    </collision>
+  </link>
+  <link name="realsense">
+    <visual>
+      <geometry>
+        <mesh filename="package://roomba_description/meshes/d435.stl" />
+      </geometry>
+    </visual>
+  </link>
+  <joint name="realsense_to_base_link" type="fixed">
+    <origin xyz="0.05 -0.033 0.045" rpy="0 0 0"/>
+    <parent link="lidar_base"/>
+    <child link="realsense"/>
+  </joint>
+  <joint name="rplidar_to_base_link" type="fixed">
+    <origin xyz="0.05 -0.033 0.045" rpy="0 0 0"/>
+    <parent link="lidar_base"/>
+    <child link="rplidar"/>
+  </joint>
+  <link name="laser"/>
+  <joint name="laser_to_rplidar" type="fixed">
+    <origin xyz="-0.035 0.0 0.045" rpy="0 0 3.14159"/>
+    <parent link="rplidar"/>
+    <child link="laser"/>
+  </joint>
+  <!--
+  <link name="mobile_battery">
+    <inertial>
+      <origin xyz="0 0 0" rpy="0 0 0"/>
+      <mass value="0.680389"/>
+      <inertia ixx="100"  ixy="0"  ixz="0" iyy="100" iyz="0" izz="100" />
+    </inertial>
+    <visual>
+      <origin xyz="0 0 0" rpy="0 0 0" />
+      <geometry>
+        <box size="0.06 0.1 0.02" />
+      </geometry>
+      <material name="white">
+          <color rgba="1.0 1.0 1.0 1.0"/>
+      </material>
+    </visual>
+    <collision>
+      <origin xyz="0 0 0" rpy="0 0 0" />
+      <geometry>
+        <box size="0.06 0.1 0.02" />
+      </geometry>
+    </collision>
+  </link>
+  <joint name="mobile_battery_to_base_link" type="fixed">
+    <origin xyz="0.0 0.0 0.09" rpy="0 1.570796 0"/>
+    <parent link="base_link"/>
+    <child link="mobile_battery"/>
+  </joint>
+  <link name="jetson_nano">
+    <inertial>
+      <origin xyz="0 0 0" rpy="0 0 0"/>
+      <mass value="1.548"/>
+      <inertia ixx="100"  ixy="0"  ixz="0" iyy="100" iyz="0" izz="100" />
+    </inertial>
+    <visual>
+      <origin xyz="0 0 0" rpy="0 0 0" />
+      <geometry>
+        <box size="0.105 0.105 0.065" />
+      </geometry>
+      <material name="grey"/>
+    </visual>
+    <collision>
+      <origin xyz="0 0 0" rpy="0 0 0" />
+      <geometry>
+        <box size="0.105 0.105 0.065" />
+      </geometry>
+    </collision>
+  </link>
+  <joint name="jetson_nano_to_base_link" type="fixed">
+    <origin xyz="-0.1 0 0.09" rpy="0 0 0"/>
+    <parent link="base_link"/>
+    <child link="jetson_nano"/>
+  </joint>
+  -->
 </robot>

Commit message: update rqlidar urdf

File: catkin_ws/src/roomba/roomba_description/urdf/roomba.urdf.xacro (robot description, xacro)
@@ -76,5 +76,5 @@
   <link name="laser"/>
   <joint name="laser_to_rplidar" type="fixed">
-    <origin xyz="-0.035 0.0 0.045" rpy="0 0 3.14159"/>
+    <origin xyz="-0.035 0.0 0.045" rpy="0 0 0"/>
     <parent link="rplidar"/>
     <child link="laser"/>

Commit message: change urdf

File: catkin_ws/src/roomba/roomba_description/urdf/roomba.urdf.xacro (robot description, xacro)
@@ -29,5 +29,5 @@
   </link>
   <joint name="lidar_base_to_base_link" type="fixed">
-    <origin xyz="-0.08 0 0.09" rpy="0 0 0"/>
+    <origin xyz="0.08 0 0.09" rpy="0 0 0"/>
     <parent link="base_link"/>
     <child link="lidar_base"/>

Commit message: change lidar

File: catkin_ws/src/roomba/roomba_description/urdf/roomba.urdf.xacro (robot description, xacro)
@@ -76,5 +76,5 @@
   <link name="laser"/>
   <joint name="laser_to_rplidar" type="fixed">
-    <origin xyz="-0.035 0.0 0.045" rpy="0 0 0"/>
+    <origin xyz="-0.035 0.03 0.03" rpy="0 0 0"/>
     <parent link="rplidar"/>
     <child link="laser"/>

Commit message: add

File: catkin_ws/src/roomba/roomba_description/urdf/roomba.urdf.xacro (robot description, xacro)
@@ -67,5 +67,5 @@
     <origin xyz="0.05 -0.033 0.045" rpy="0 0 0"/>
     <parent link="lidar_base"/>
-    <child link="realsense"/>
+    <child link="camera_link"/>
   </joint>
   <joint name="rplidar_to_base_link" type="fixed">

Commit message: add

File: catkin_ws/src/roomba/roomba_description/urdf/roomba.urdf.xacro (robot description, xacro)
@@ -67,5 +67,5 @@
     <origin xyz="0.05 -0.033 0.045" rpy="0 0 0"/>
     <parent link="lidar_base"/>
-    <child link="camera_link"/>
+    <child link="realsense"/>
   </joint>
   <joint name="rplidar_to_base_link" type="fixed">

Commit message: define camera_link in urdf

File: catkin_ws/src/roomba/roomba_description/urdf/roomba.urdf.xacro (robot description, xacro)
@@ -69,4 +69,10 @@
     <child link="realsense"/>
   </joint>
+  <link name="camera_link">
+  <joint name="camera_link_to_realsense" type="fixed">
+    <origin xyz="0 0 0" rpy="0 0 0"/>
+    <parent link="realsense"/>
+    <child link="camera_link"/>
+  </joint>
   <joint name="rplidar_to_base_link" type="fixed">
     <origin xyz="0.05 -0.033 0.045" rpy="0 0 0"/>

Commit message: fix typo

File: catkin_ws/src/roomba/roomba_description/urdf/roomba.urdf.xacro (robot description, xacro)
@@ -69,5 +69,5 @@
     <child link="realsense"/>
   </joint>
-  <link name="camera_link">
+  <link name="camera_link"/>
   <joint name="camera_link_to_realsense" type="fixed">
     <origin xyz="0 0 0" rpy="0 0 0"/>
